File: Runout8x.kicad_pcb (KiCad board)
At the start: 2 copper layers, 22.9 x 129.5 mm, 19 parts, among them M1 Fan_Tacho, M2 Fan_Tacho_PWM, U1 XIAO-RP2040-SMD

Commit message: Routing cleanup
Routing:
- net Net-(M2-Tacho): track 21.9 -> 9.46 mm
- net /Channel1/PWR: track 122.1 -> 130.2 mm
- net /Channel8/SIG: track 63.4 -> 69.7 mm
- net /Channel1/GND: track 1.42 -> 5.89 mm
- net /Channel7/SIG: track 51.1 -> 54.2 mm
- net /Channel2/SIG: track 48.8 -> 47.7 mm
- net /Channel1/SIG: track 62.6 -> 61.5 mm
- net /Channel6/SIG: track 38.9 -> 39.7 mm
- net Net-(M1-+): track 28.8 -> 29.3 mm
Other:
- board text added: "8 WAY FILAMENT RUNOUT SENSOR Rev 0.1"
- board text added: "Molot Makes Things"
- board text added: "WayWayWay"
